File: rgb_led_cube.kicad_pcb (KiCad board)
At the start: 2 copper layers, 279.4 x 254 mm, 90 parts, among them Q1 IRLML6401TRPBF, Q10 MMBT2222A-TP, Q11 IRLML6401TRPBF, Q12 MMBT2222A-TP, Q13 IRLML6401TRPBF, Q14 MMBT2222A-TP, Q15 IRLML6401TRPBF, Q16 MMBT2222A-TP, Q2 MMBT2222A-TP, Q3 IRLML6401TRPBF, Q4 MMBT2222A-TP, Q5 IRLML6401TRPBF, Q6 MMBT2222A-TP, Q7 IRLML6401TRPBF, Q8 MMBT2222A-TP, Q9 IRLML6401TRPBF, U1 TLC59711PWPR, U10 TLC59711PWPR, U11 TLC59711PWPR, U12 TLC59711PWPR, U13 TLC59711PWPR, U14 TLC59711PWPR, U15 TLC59711PWPR, U16 TLC59711PWPR, U2 TLC59711PWPR, U3 TLC59711PWPR, U4 TLC59711PWPR, U5 TLC59711PWPR, U6 TLC59711PWPR, U7 TLC59711PWPR, U8 TLC59711PWPR, U9 TLC59711PWPR

Commit message: Arrange TLC with resistors and capacitors
Parts:
- moved DS1 551.2 mm to (140.7, 167.4)
- moved Q5 434.2 mm to (303.5, 314.3)
- moved Q1 434.2 mm to (287.5, 330.8)
- moved Q10 434.2 mm to (308.8, 315.4)
- moved Q11 434.2 mm to (316.3, 303.3)
- moved Q12 434.2 mm to (327.0, 292.3)
- moved Q13 434.2 mm to (171.6, 287.2)
- moved Q14 434.2 mm to (166.9, 292.1)
- moved Q15 434.2 mm to (286.4, 339.6)
- moved Q16 434.2 mm to (171.6, 292.1)
- moved Q2 434.2 mm to (166.9, 287.2)
- moved Q3 434.2 mm to (320.6, 293.4)
- moved Q4 434.2 mm to (312.1, 304.4)
- moved Q6 434.2 mm to (294.9, 324.2)
- moved Q7 434.2 mm to (288.5, 337.4)
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
Commit message: Update components placement
Parts:
- moved R17 264.7 mm to (259.1, 59.9), turned to 180 degrees
- moved Q1 260.5 mm to (259.1, 71.9), turned to 270 degrees
- moved R18 255.1 mm to (257.8, 67.6), turned to 90 degrees
- moved R19 254.0 mm to (260.1, 67.6), turned to 90 degrees
- moved Q2 242.2 mm to (259.1, 63.2), turned to 270 degrees
- moved R20 233.3 mm to (259.1, 87.9), turned to 180 degrees
- moved R21 223.8 mm to (257.8, 95.5), turned to 90 degrees
- moved R22 222.7 mm to (260.1, 95.5), turned to 90 degrees
- moved Q4 219.7 mm to (259.1, 91.2), turned to 270 degrees
- moved Q6 208.2 mm to (259.1, 119.1), turned to 270 degrees
- moved R23 207.9 mm to (259.1, 115.8), turned to 180 degrees
- moved Q3 203.1 mm to (259.1, 99.8), turned to 270 degrees
- moved Q5 191.8 mm to (259.1, 127.8), turned to 270 degrees
- moved R24 185.3 mm to (257.8, 123.4), turned to 90 degrees
- moved Q7 184.1 mm to (259.1, 155.7), turned to 270 degrees
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Connections:
- R17 pad 2: Net-(R17-Pad2) -> Net-(CNTL1-Pad15)
- R20 pad 2: Net-(R20-Pad2) -> Net-(CNTL1-Pad13)
- R23 pad 2: Net-(R23-Pad2) -> Net-(CNTL1-Pad12)
- R26 pad 2: Net-(R26-Pad2) -> Net-(CNTL1-Pad11)
- R29 pad 2: Net-(R29-Pad2) -> Net-(CNTL1-Pad10)
- R32 pad 2: Net-(R32-Pad2) -> Net-(CNTL1-Pad9)
- R35 pad 2: Net-(R35-Pad2) -> Net-(CNTL1-Pad8)
- R38 pad 2: Net-(R38-Pad2) -> Net-(CNTL1-Pad7)
Routing:
- net Net-(Q2-Pad3): track 0.00 -> 4.54 mm
- net VCC: track 0.00 -> 2.38 mm
- net Net-(Q2-Pad1): track 0.00 -> 2.28 mm
- net Net-(Q1-Pad1): track 0.00 -> 2.27 mm
Other:
- board size 279.4 x 254 mm -> 246.4 x 238.8 mm

Commit message: Route ICs
Parts:
- moved R38 38.2 mm to (259.1, 265.4), turned to 0 degrees
- moved Q16 31.7 mm to (259.1, 262.1), turned to 90 degrees
- moved R39 23.9 mm to (260.4, 257.8), turned to 270 degrees
- moved R40 22.8 mm to (258.1, 257.8), turned to 270 degrees
- moved Q15 14.9 mm to (259.1, 253.5), turned to 90 degrees
- moved C16 10.2 mm to (147.1, 266.2)
- moved C4 10.2 mm to (147.1, 98.6)
- moved C6 10.2 mm to (147.1, 126.5)
- moved R2 10.2 mm to (147.1, 66.5)
- moved C10 10.2 mm to (147.1, 182.4)
- moved C14 10.2 mm to (147.1, 238.3)
- moved C2 10.2 mm to (147.1, 70.6)
- moved C8 10.2 mm to (147.1, 154.4)
- moved R10 10.2 mm to (147.1, 178.3)
- moved R14 10.2 mm to (147.1, 234.2)
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Connections:
- CNTL1 pad 18: GND -> Net-(CNTL1-Pad18)
Routing:
- net VCC: track 2.38 -> 44.9 mm
- net Net-(U8-Pad12): track 0.00 -> 9.64 mm
- net Net-(U8-Pad11): track 0.00 -> 9.64 mm
- net Net-(U10-Pad12): track 0.00 -> 9.64 mm
- net Net-(U10-Pad11): track 0.00 -> 9.64 mm
- net Net-(U6-Pad12): track 0.00 -> 9.64 mm
- net Net-(U6-Pad11): track 0.00 -> 9.64 mm
- net Net-(U4-Pad12): track 0.00 -> 9.64 mm
- net Net-(U4-Pad11): track 0.00 -> 9.64 mm
- net Net-(U2-Pad12): track 0.00 -> 9.64 mm
- net Net-(U2-Pad11): track 0.00 -> 9.64 mm
- net Net-(U14-Pad12): track 0.00 -> 9.64 mm
- net Net-(U14-Pad11): track 0.00 -> 9.64 mm
- net Net-(U12-Pad12): track 0.00 -> 9.64 mm
- net Net-(U12-Pad11): track 0.00 -> 9.64 mm
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
Commit message: Route pcb
Parts:
- Q1, Q10, Q11, Q12, Q13, Q14, Q15, Q16, Q2, Q3, Q4, Q5, Q6, Q7, Q8, Q9: footprint digikey-footprints:SOT-23-3 -> Package_TO_SOT_SMD:SOT-23
- U1, U10, U11, U12, U13, U14, U15, U16, U2, U3, U4, U5, U6, U7, U8, U9: footprint digikey-footprints:TSSOP-20-1EP_W4.4mm -> Package_SO:HTSSOP-20-1EP_4.4x6.5mm_P0.65mm_EP3.4x6.5mm_Mask2.75x3.43mm_ThermalVias
- moved CNTL1 149.2 mm to (49.0, 87.7), turned to 270 degrees
- moved R5 61.8 mm to (85.7, 102.6), turned to 180 degrees
- moved R1 61.8 mm to (85.7, 46.7), turned to 180 degrees
- moved R11 61.8 mm to (85.7, 186.4), turned to 180 degrees
- moved R13 61.8 mm to (85.7, 214.3), turned to 180 degrees
- moved R15 61.8 mm to (85.7, 242.3), turned to 180 degrees
- moved R3 61.8 mm to (85.7, 74.6), turned to 180 degrees
- moved R7 61.8 mm to (85.7, 130.5), turned to 180 degrees
- moved R9 61.8 mm to (85.7, 158.4), turned to 180 degrees
- moved U10 59.7 mm to (199.5, 163.2), turned to 0 degrees
- moved U12 59.7 mm to (199.5, 191.2), turned to 0 degrees
- moved U14 59.7 mm to (199.5, 219.1), turned to 0 degrees
- moved U16 59.7 mm to (199.5, 247.1), turned to 0 degrees
- moved U2 59.7 mm to (199.5, 51.5), turned to 0 degrees
- moved U4 59.7 mm to (199.5, 79.4), turned to 0 degrees
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Routing:
- net VCC: track 44.9 -> 975.1 mm, vias 0 -> 25
- net Net-(CNTL1-Pad7): track 0.00 -> 410.9 mm, vias 0 -> 2
- net Net-(CNTL1-Pad8): track 0.00 -> 365.5 mm, vias 0 -> 2
- net Net-(CNTL1-Pad9): track 0.00 -> 338.2 mm, vias 0 -> 2
- net Net-(CNTL1-Pad10): track 0.00 -> 314.7 mm, vias 0 -> 2
- net Net-(CNTL1-Pad11): track 0.00 -> 285.5 mm, vias 0 -> 2
- net Net-(CNTL1-Pad12): track 0.00 -> 265.7 mm, vias 0 -> 2
- net Net-(CNTL1-Pad15): track 0.00 -> 242.3 mm, vias 0 -> 2
- net Net-(CNTL1-Pad13): track 0.00 -> 235.1 mm, vias 0 -> 2
- net Net-(U14-Pad12): track 9.64 -> 151.3 mm, vias 0 -> 4
- net Net-(U2-Pad12): track 9.64 -> 150.1 mm, vias 0 -> 4
- net Net-(U8-Pad12): track 9.64 -> 150.0 mm, vias 0 -> 4
- net Net-(U4-Pad12): track 9.64 -> 149.8 mm, vias 0 -> 4
- net Net-(U6-Pad12): track 9.64 -> 149.8 mm, vias 0 -> 4
- net Net-(U12-Pad12): track 9.64 -> 149.7 mm, vias 0 -> 4
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- added copper zone on F.Cu, net GND

Commit message: Connect unused header pins to GND
Connections:
- CNTL1 pad 39: Net-(CNTL1-Pad39) -> GND
- CNTL1 pad 40: Net-(CNTL1-Pad40) -> GND
